File: HARDWARE/DESIGN/esp32_control-board/esp32cb_main.kicad_sch (KiCad schematic)
At the start: 12 parts, among them SW301 espM_Reset, SW302 espM_Boot, U1 ESP32-S3-WROOM-1

Commit message: 60707 - schematics and readme updated, preliminary PCB-layout prepared
Parts:
- removed R306, R307: 2k2, Resistor_SMD:R_0603_1608Metric, symbol Device:R
- added C314, C315: 1u, Capacitor_SMD:C_0603_1608Metric, symbol Device:C
- added J10: ESP32-Prog, Connector_PinHeader_2.54mm:PinHeader_1x04_P2.54mm_Vertical, symbol Connector:Screw_Terminal_01x04
- added J11: RFID-module1, Connector_JST:JST_PH_B8B-PH-K_1x08_P2.00mm_Vertical, symbol Connector:Screw_Terminal_01x08
- added J12: RFID-module2, Connector_JST:JST_PH_B8B-PH-K_1x08_P2.00mm_Vertical, symbol Connector:Screw_Terminal_01x08
- added R336, R337: 5k1, Resistor_SMD:R_0603_1608Metric, symbol Device:R
- SW301: value espM_Reset -> Reset
- SW302: value espM_Boot -> Boot
Connections:
- net espM_Boot is gone; now on net esp_Boot: R305.2, SW302.1
- net espM_Reset is gone; now on net esp_Reset: C303.2, R304.2, SW301.1
- net +3V3: now also C314.1, C315.1, J10.1 (Pin_1), J11.8 (Pin_8), J12.8 (Pin_8), R336.2, R337.2
- net GND: now also C314.2, C315.2, J10.4 (Pin_4), J11.6 (Pin_6), J12.6 (Pin_6)
- net I2C_scl: now also R337.1
- net I2C_sda: now also R336.1
- net SPI_miso: now also J11.4 (Pin_4), J12.4 (Pin_4)
- net SPI_mosi: now also J11.3 (Pin_3), J12.3 (Pin_3)
- net SPI_sck: now also J11.2 (Pin_2), J12.2 (Pin_2)
- net esp_Boot: now reaches U1.27 (IO0)
- net esp_Reset: now reaches U1.3 (EN)
- net esp_Rx: now reaches U1.36 (RXD0)
- net esp_Rx: now also J10.2 (Pin_2)
- net esp_Tx: now reaches U1.37 (TXD0)
- net esp_Tx: now also J10.3 (Pin_3)
- net SPI_cs renamed SPI_cs1
- net SPI_cs1: now also J11.1 (Pin_1)
- new net RFID1_irq: J11.5 (Pin_5)
- new net RFID1_reset: J11.7 (Pin_7)
- new net RFID2_irq: J12.5 (Pin_5)
- new net RFID2_reset: J12.7 (Pin_7)
- new net SPI_cs2: J12.1 (Pin_1)
Other:
- title: (none) -> ESP32-based Control Board
- moved on the sheet: C303, R304, R305, SW301, SW302
