File: HARDWARE/DESIGN/esp32_control-board/esp32cb_inputs.kicad_sch (KiCad schematic)
At the start: 56 parts, among them J1 Lock1, J2 Lock2, J3 Lock3, J4 Lock4, J5 Lock5, J6 Lock6, J7 Lock7, J8 Lock8, U10 PC817, U11 PC817, U12 PC817, U13 PC817, U14 PC817, U15 PC817, U16 PC817, U5 PC817

Commit message: 60714 - one of two I2C-mux ICs was removed, PCB-layout finished, start tracing
Parts:
- added JP409, JP410, JP411, JP412, JP413, JP414, JP415, JP416: 12V-to-COM, Jumper:SolderJumper-2_P1.3mm_Bridged_RoundedPad1.0x1.5mm, symbol Jumper:Jumper_2_Bridged
- renumbered C306 to C401, C307 to C402, C308 to C403, C309 to C404, C310 to C405, C311 to C406, C312 to C407, C313 to C408, D4 to D401, D5 to D402, D6 to D403, D7 to D404, D8 to D405, D9 to D406, D10 to D407, D11 to D408, J1 to J401, J2 to J402, J3 to J403, J4 to J404, J5 to J405, J6 to J406, J7 to J407, J8 to J408, JP2 to JP401, JP3 to JP402, JP4 to JP403, JP5 to JP404, JP6 to JP405, JP7 to JP406, JP8 to JP407, JP9 to JP408, R2 to R401, R3 to R402, R4 to R403, R5 to R404, R327 to R405, R329 to R406, R330 to R407, R331 to R408, R6 to R409, R7 to R410, R8 to R411, R9 to R412, R332 to R413, R333 to R414, R334 to R415, R335 to R416, U5 to U401, U10 to U402, U11 to U403, U12 to U404, U13 to U405, U14 to U406, U15 to U407, U16 to U408
Connections:
- net +12V: now also JP409.1 (A), JP410.1 (A), JP411.1 (A), JP412.1 (A), JP413.1 (A), JP414.1 (A), JP415.1 (A), JP416.1 (A); no longer J401.4 (Pin_4), J402.4 (Pin_4), J403.4 (Pin_4), J404.4 (Pin_4), J405.4 (Pin_4), J406.4 (Pin_4), J407.4 (Pin_4), J408.4 (Pin_4)
- new net SWITCH1-COM: J401.4 (Pin_4), JP409.2 (B)
- new net SWITCH2-COM: J402.4 (Pin_4), JP410.2 (B)
- new net SWITCH3-COM: J403.4 (Pin_4), JP411.2 (B)
- new net SWITCH4-COM: J404.4 (Pin_4), JP412.2 (B)
- new net SWITCH5-COM: J405.4 (Pin_4), JP413.2 (B)
- new net SWITCH6-COM: J406.4 (Pin_4), JP414.2 (B)
- new net SWITCH7-COM: J407.4 (Pin_4), JP415.2 (B)
- new net SWITCH8-COM: J408.4 (Pin_4), JP416.2 (B)
