File: HARDWARE/DESIGN/esp32_control-board/esp32cb_locks.kicad_sch (KiCad schematic)
At the start: 9 parts, among them J409 Lock1, J410 Lock2, Q401 AO3401A, U409 PC817

Commit message: 60825 - Schematic update and PCB-layout started
Parts:
- removed JP417: Switch State Selector, Jumper:SolderJumper-3_P1.3mm_Bridged12_RoundedPad1.0x1.5mm, symbol Jumper:Jumper_3_Bridged12
- removed R418: 10k, Resistor_SMD:R_0603_1608Metric, symbol Device:R
- added C410, C411, C412: 1n, Capacitor_SMD:C_0603_1608Metric, symbol Device:C
- added D106, D107, D108, D109: XL-1608UOC-06, LED_SMD:LED_0603_1608Metric, symbol Device:LED
- added D410, D411, D412: 1N4148W, Diode_SMD:D_SOD-123, symbol Diode:1N4148W
- added Q402, Q403, Q405: BSS138, Package_TO_SOT_SMD:SOT-23, symbol Transistor_FET:BSS138
- added Q404: AO3401A, Package_TO_SOT_SMD:SOT-23, symbol Transistor_FET:AO3401A
- added Q406: DMP6180SK3-13, Package_TO_SOT_SMD:TO-252-2, symbol Transistor_FET:AO3401A
- added R105, R107, R113, R115, R116, R117, R118, R119, R133, R134: 12k, Resistor_SMD:R_0603_1608Metric, symbol Device:R
- added R106, R114: 27k, Resistor_SMD:R_0603_1608Metric, symbol Device:R
- added R111, R112, R124: 120, Resistor_SMD:R_0603_1608Metric, symbol Device:R
- added R419, R420, R421: 1k, Resistor_SMD:R_0603_1608Metric, symbol Device:R
- added U410, U411, U412: PC817, Package_DIP:DIP-4_W7.62mm_SMDSocket_SmallPads, symbol Isolator:PC817
- Q401: LCSC (none) -> C2938368; Manufacturer (none) -> GOODWORK; Package (none) -> SOT-23
- R417: value 1k2 -> 1k; LCSC C114605 -> (none); LCSC part (none) -> C21190; Manufacturer YAGEO -> UNI-ROYAL(Uniroyal Elec)
Connections:
- net ctrl_LOCK1 is gone; now on net ctrl_LOCK1_12V: J409.3 (Pin_3)
- net +12V: now also Q401.2 (S), Q404.2 (S), Q406.2 (S), R106.2, R114.2, R134.1
- net +3V3: now also R116.1, R117.1, R118.1, R119.1
- net GND: now also C410.1, C411.1, C412.1, D410.2 (A), D411.2 (A), D412.2 (A), Q402.2 (S), Q403.2 (S), Q405.2 (S), R105.2, R113.2, R133.2, U410.2, U411.2, U412.2
- net GND_MCU: now also U410.3, U411.3, U412.3
- net at C409.2: now also D409.1 (K), R417.2, D106.2 (A); no longer R417.1
- net at Q401.1 (G): now also R107.2
- net ctrl_LOCK1_12V: now reaches Q401.3 (D)
- net LOCK1_signal renamed sens_LOCK1_latch_3V3
- net sens_LOCK1_latch_3V3: now also R116.2
- net ctrl_LOCK2 renamed ctrl_LOCK2_12V
- net ctrl_LOCK2_12V: now also Q404.3 (D)
- net sens_DOOR_LOCK1 renamed sens_LOCK1_door_12V
- net sens_LOCK1_door_12V: now also R419.1
- net sens_DOOR_LOCK2 renamed sens_LOCK2_door_12V
- net sens_LOCK2_door_12V: now also R421.1
- net sens_LATCH_LOCK1 renamed sens_LOCK1_latch_12V
- net sens_LOCK1_latch_12V: now also R417.1
- net sens_LATCH_LOCK2 renamed sens_LOCK2_latch_12V
- net sens_LOCK2_latch_12V: now also R420.1
- new net: C412.2, D109.2 (A), D412.1 (K), R421.2
- new net: Q404.1 (G), R115.2
- new net: C411.2, D108.2 (A), D411.1 (K), R420.2
- new net: D109.1 (K), U412.1
- new net: Q402.1 (G), R105.1, R111.2
- new net: Q402.3 (D), R106.1, R107.1
- new net: D108.1 (K), U411.1
- new net: D107.1 (K), U410.1
- new net: C410.2, D107.2 (A), D410.1 (K), R419.2
- new net: Q405.1 (G), R124.2, R133.1
- new net: D106.1 (K), U409.1
- new net: Q403.3 (D), R114.1, R115.1
- new net: Q405.3 (D), Q406.1 (G), R134.2
- new net: Q403.1 (G), R112.2, R113.1
- new net ctrl_LAMP_12V: Q406.3 (D)
- new net ctrl_LAMP_3V3: R124.1
- new net ctrl_LOCK1_3V3: R111.1
- new net ctrl_LOCK2_3V3: R112.1
- new net sens_LOCK1_door_3V3: R117.2, U410.4
- new net sens_LOCK2_door_3V3: R119.2, U412.4
- new net sens_LOCK2_latch_3V3: R118.2, U411.4
Other:
- note added: "8.7mA at 12V-input"
- note added: "Lamp control circuit"
- note added: "Lock1 sensors' processing circuits"
- note added: "Lock2 sensors' processing circuits"
- note added: "Locks' connectors"
- note added: "Locks' control circuits"
- note added: "Vgs-limitation"
- moved on the sheet: C409, D409, J409, J410, Q401, U409

Commit message: 60905 - fuse-holder replaced, led-strip connector added
Parts:
- Q405, Q406: now not fitted; now left out of the parts list
- R124, R133, R134: now not fitted
Changed lines of the file:
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@@
 		(exclude_from_sim no)
 		(in_bom no)
-		(on_board yes)
-		(in_pos_files yes)
-		(dnp no)
+		(on_board no)
+		(in_pos_files no)
+		(dnp yes)
 		(property "Reference" "R133"
 			(at 179.832 467.868 0)
@@
 		(exclude_from_sim no)
 		(in_bom no)
-		(on_board yes)
-		(in_pos_files yes)
-		(dnp no)
+		(on_board no)
+		(in_pos_files no)
+		(dnp yes)
 		(property "Reference" "R134"
 			(at 200.152 441.198 0)
@@
 		(body_style 1)
 		(exclude_from_sim no)
-		(in_bom yes)
-		(on_board yes)
-		(in_pos_files yes)
-		(dnp no)
+		(in_bom no)
+		(on_board no)
+		(in_pos_files no)
+		(dnp yes)
 		(property "Reference" "Q406"
 			(at 223.52 429.514 90)
@@
 		(exclude_from_sim no)
 		(in_bom no)
-		(on_board yes)
-		(in_pos_files yes)
-		(dnp no)
+		(on_board no)
+		(in_pos_files no)
+		(dnp yes)
 		(property "Reference" "R124"
 			(at 163.83 457.962 90)
@@
 		(body_style 1)
 		(exclude_from_sim no)
-		(in_bom yes)
-		(on_board yes)
-		(in_pos_files yes)
-		(dnp no)
+		(in_bom no)
+		(on_board no)
+		(in_pos_files no)
+		(dnp yes)
 		(property "Reference" "Q405"
 			(at 201.168 459.74 0)
