File: HARDWARE/DESIGN/esp32_control-board/esp32cb_can.kicad_sch (KiCad schematic)
At the start: 8 parts, among them J4 Termination, J401 B3B-PH-K-K(LF)(SN), U6 TCAN330

Commit message: 60828 - Schematic updated, preliminary PCB-layout done
Parts:
- FL1: footprint FOOTPRINTS:C76584_IND-SMD_4P-L4.5-W3.2-TL -> (FOOTPRINTS):C76584_IND-SMD_4P-L4.5-W3.2-TL
- J401: value B3B-PH-K-K(LF)(SN) -> CAN; footprint Connector_JST:JST_PH_B3B-PH-K_1x03_P2.00mm_Vertical -> Connector_JST:JST_PH_S3B-PH-K_1x03_P2.00mm_Horizontal; LCSC C5305733 -> (none)
Changed lines of the file:
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@@
 	(title_block
 		(title "ESP32-based Control Board")
-		(date "2026-08-25")
+		(date "2026-08-28")
 		(rev "2a")
 	)
@@
 			)
 		)
-		(property "Value" "B3B-PH-K-K(LF)(SN)"
+		(property "Value" "CAN"
 			(at 300.99 190.5 0)
 			(show_name no)
@@
 			)
 		)
-		(property "Footprint" "Connector_JST:JST_PH_B3B-PH-K_1x03_P2.00mm_Vertical"
+		(property "Footprint" "Connector_JST:JST_PH_S3B-PH-K_1x03_P2.00mm_Horizontal"
 			(at 303.53 191.77 0)
 			(hide yes)
@@
 			)
 		)
-		(property "LCSC" "C5305733"
+		(property "LCSC" ""
 			(at 303.53 191.77 0)
 			(hide yes)
@@
 			)
 		)
-		(property "Footprint" "FOOTPRINTS:C76584_IND-SMD_4P-L4.5-W3.2-TL"
+		(property "Footprint" "(FOOTPRINTS):C76584_IND-SMD_4P-L4.5-W3.2-TL"
 			(at 114.3 76.2 0)
 			(hide yes)

Commit message: 60908 - PCB-layout updated
Connections:
- net CAN+_conn.: now also J401.3 (Pin_3); no longer J401.1 (Pin_1)
- net GND: now also J401.1 (Pin_1); no longer J401.3 (Pin_3)
Other:
- moved on the sheet: J401
Changed lines of the file:
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@@
 	(symbol
 		(lib_id "Connector_Generic:Conn_01x03")
-		(at 303.53 191.77 0)
-		(mirror y)
+		(at 303.53 191.77 180)
 		(unit 1)
 		(body_style 1)
@@
 		(dnp no)
 		(property "Reference" "J401"
-			(at 300.99 187.96 0)
+			(at 300.99 195.58 0)
 			(show_name no)
 			(do_not_autoplace no)
@@
 		)
 		(property "Value" "CAN"
-			(at 300.99 190.5 0)
+			(at 300.99 193.04 0)
 			(show_name no)
 			(do_not_autoplace no)
@@
 		)
 		(property "Package" "PH-2.0"
-			(at 300.99 195.326 0)
+			(at 300.99 188.214 0)
 			(show_name no)
 			(do_not_autoplace no)
@@
 		)
 		(property "Property" "Black"
-			(at 300.99 193.0401 0)
+			(at 300.99 190.4999 0)
 			(show_name no)
 			(do_not_autoplace no)
