File: HARDWARE/DESIGN/esp32_control-board/esp32cb_power.kicad_sch (KiCad schematic)
At the start: 32 parts, among them J101 Power-in, Q101 AO4407C, Q102 DMP3013SFV-7, U101 LM63615DQDRRRQ1, U102 AMS1117-3.3

Commit message: 60911 - PCB-layout updated
Parts:
- C109: now not fitted; now left out of the parts list
Changed lines of the file:
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@@
 		(body_style 1)
 		(exclude_from_sim no)
-		(in_bom yes)
-		(on_board yes)
-		(in_pos_files yes)
-		(dnp no)
+		(in_bom no)
+		(on_board no)
+		(in_pos_files no)
+		(dnp yes)
 		(property "Reference" "C109"
 			(at 228.346 193.294 0)
@@
 			(show_name no)
 			(do_not_autoplace no)
+			(effects
+				(font
+					(size 1.27 1.27)
+				)
+			)
+		)
+		(property "LCSC" ""
+			(at 224.79 196.85 0)
+			(hide yes)
+			(show_name no)
+			(do_not_autoplace no)
